Commit message: update

File: mycobot_description/robots/mycobot_with_gripper_camera.urdf.xacro (robot description, xacro)
@@ -16,5 +16,5 @@
   <!-- Mycobot arm -->
   <xacro:mycobot_arm parent="world">
-    <origin xyz="0 0 0" rpy="0 0 0" />
+    <origin xyz="0 0 0.95" rpy="0 0 0" />
   </xacro:mycobot_arm>
   <!-- Mycobot gripper -->
@@ -23,6 +23,6 @@
   </xacro:mycobot_gripper>
   <!-- D435 camera -->
-  <xacro:sensor_d435 name="camera" topics_ns="camera" parent="world" publish_pointcloud="true">
-    <origin xyz="-0.5 0 0.5" rpy="0 0 0" />
+  <xacro:sensor_d435 name="d435_camera" topics_ns="d435_camera" parent="world" publish_pointcloud="true">
+    <origin xyz="0 0.5 1.5" rpy="0 ${pi/2} 0" />
   </xacro:sensor_d435>
 </robot>

File: mycobot_moveit_config/config/gazebo_mycobot.urdf (robot description, URDF)
Before this commit: robot mycobot, 25 links, 24 joints
Links:
- removed link camera_bottom_screw_frame
- removed link camera_color_frame
- removed link camera_color_optical_frame
- removed link camera_depth_frame
- removed link camera_depth_optical_frame
- removed link camera_left_ir_frame
- removed link camera_left_ir_optical_frame
- removed link camera_link
- removed link camera_right_ir_frame
- removed link camera_right_ir_optical_frame
- added link d435_camera_bottom_screw_frame
- added link d435_camera_color_frame
- added link d435_camera_color_optical_frame
- added link d435_camera_depth_frame
- added link d435_camera_depth_optical_frame
- added link d435_camera_left_ir_frame
- added link d435_camera_left_ir_optical_frame
- added link d435_camera_link, mass 0.564; collision box size=0.02505 0.09 0.025; visual mesh filename=package://mycobot_description/meshes/camera/d435.dae
- added link d435_camera_right_ir_frame
- added link d435_camera_right_ir_optical_frame
Joints:
- removed joint camera_color_joint
- removed joint camera_color_optical_joint
- removed joint camera_depth_joint
- removed joint camera_depth_optical_joint
- removed joint camera_joint
- removed joint camera_left_ir_joint
- removed joint camera_left_ir_optical_joint
- removed joint camera_link_joint
- removed joint camera_right_ir_joint
- removed joint camera_right_ir_optical_joint
- added joint d435_camera_color_joint: type fixed, parent d435_camera_depth_frame, child d435_camera_color_frame, origin xyz=0 0.015 0 rpy=0 0 0
- added joint d435_camera_color_optical_joint: type fixed, parent d435_camera_color_frame, child d435_camera_color_optical_frame, origin xyz=0 0 0 rpy=-1.5707963267948966 0 -1.5707963267948966
- added joint d435_camera_depth_joint: type fixed, parent d435_camera_link, child d435_camera_depth_frame, origin xyz=0 0 0 rpy=0 0 0
- added joint d435_camera_depth_optical_joint: type fixed, parent d435_camera_depth_frame, child d435_camera_depth_optical_frame, origin xyz=0 0 0 rpy=-1.5707963267948966 0 -1.5707963267948966
- added joint d435_camera_joint: type fixed, parent world, child d435_camera_bottom_screw_frame, origin xyz=0 0.5 1.5 rpy=0 1.5707963267948966 0
- added joint d435_camera_left_ir_joint: type fixed, parent d435_camera_depth_frame, child d435_camera_left_ir_frame, origin xyz=0 0.0 0 rpy=0 0 0
- added joint d435_camera_left_ir_optical_joint: type fixed, parent d435_camera_left_ir_frame, child d435_camera_left_ir_optical_frame, origin xyz=0 0 0 rpy=-1.5707963267948966 0 -1.5707963267948966
- added joint d435_camera_link_joint: type fixed, parent d435_camera_bottom_screw_frame, child d435_camera_link, origin xyz=0 0.0175 0.0125 rpy=0 0 0
- added joint d435_camera_right_ir_joint: type fixed, parent d435_camera_depth_frame, child d435_camera_right_ir_frame, origin xyz=0 -0.05 0 rpy=0 0 0
- added joint d435_camera_right_ir_optical_joint: type fixed, parent d435_camera_right_ir_frame, child d435_camera_right_ir_optical_frame, origin xyz=0 0 0 rpy=-1.5707963267948966 0 -1.5707963267948966
- joint body_joint: origin xyz=0 0 0 rpy=0 0 0 -> xyz=0 0 0.95 rpy=0 0 0

Commit message: update

File: mycobot_description/robots/mycobot_with_gripper_camera.urdf.xacro (robot description, xacro)
@@ -16,5 +16,5 @@
   <!-- Mycobot arm -->
   <xacro:mycobot_arm parent="world">
-    <origin xyz="0 0 0.95" rpy="0 0 0" />
+    <origin xyz="0 0 0.95" rpy="0 0 ${pi/2}" />
   </xacro:mycobot_arm>
   <!-- Mycobot gripper -->
@@ -24,5 +24,5 @@
   <!-- D435 camera -->
   <xacro:sensor_d435 name="d435_camera" topics_ns="d435_camera" parent="world" publish_pointcloud="true">
-    <origin xyz="0 0.5 1.5" rpy="0 ${pi/2} 0" />
+    <origin xyz="0 0.5 2" rpy="0 ${pi/2} ${pi/2}" />
   </xacro:sensor_d435>
 </robot>

File: mycobot_description/urdf/arm/arm.gazebo.xacro (robot description, xacro)
@@ -14,35 +14,35 @@
 	    <mu2>${mu}</mu2>
 	    <kp>${kp}</kp>
-        <kd>${kd}</kd>
-  	</gazebo>
+      <kd>${kd}</kd>
+  </gazebo>
 	<gazebo reference="arm2_link">
 	    <mu1>${mu}</mu1>
 	    <mu2>${mu}</mu2>
 	    <kp>${kp}</kp>
-        <kd>${kd}</kd>
-  	</gazebo>
+      <kd>${kd}</kd>
+  </gazebo>
 	<gazebo reference="arm3_link">
 	    <mu1>${mu}</mu1>
 	    <mu2>${mu}</mu2>
 	    <kp>${kp}</kp>
-        <kd>${kd}</kd>
-  	</gazebo>
+      <kd>${kd}</kd>
+  </gazebo>
 	<gazebo reference="arm4_link">
 	    <mu1>${mu}</mu1>
 	    <mu2>${mu}</mu2>
 	    <kp>${kp}</kp>
-        <kd>${kd}</kd>
-  	</gazebo>
-    <gazebo reference="arm5_link">
-	    <mu1>${mu}</mu1>
-	    <mu2>${mu}</mu2>
-	    <kp>${kp}</kp>
-        <kd>${kd}</kd>
-  	</gazebo>
+      <kd>${kd}</kd>
+  </gazebo>
+  <gazebo reference="arm5_link">
+    <mu1>${mu}</mu1>
+    <mu2>${mu}</mu2>
+    <kp>${kp}</kp>
+    <kd>${kd}</kd>
+	</gazebo>
 	<gazebo reference="arm5_flange">
-	    <mu1>${mu}</mu1>
-	    <mu2>${mu}</mu2>
-	    <kp>${kp}</kp>
-        <kd>${kd}</kd>
-  	</gazebo>
+    <mu1>${mu}</mu1>
+    <mu2>${mu}</mu2>
+    <kp>${kp}</kp>
+    <kd>${kd}</kd>
+  </gazebo>
 </robot>

File: mycobot_gripper_description/urdf/gripper.gazebo.xacro (robot description, xacro)
@@ -29,12 +29,12 @@
   		parent_joint="left_outer_base_knuckle_joint" mimic_joint="left_inner_knuckle_finger_joint"
     	has_pid="true" multiplier="-1.0" max_effort="10.0" />
-  <xacro:mimic_joint_plugin_gazebo name_prefix="right_inner_base_knuckle_joint"
-		parent_joint="left_outer_base_knuckle_joint" mimic_joint="right_inner_base_knuckle_joint"
-  	has_pid="true" multiplier="-1.0" max_effort="10.0" />
-  <xacro:mimic_joint_plugin_gazebo name_prefix="right_inner_knuckle_finger_joint"
-		parent_joint="left_outer_base_knuckle_joint" mimic_joint="right_inner_knuckle_finger_joint"
-  	has_pid="true" multiplier="1.0" max_effort="10.0" />
-  <xacro:mimic_joint_plugin_gazebo name_prefix="right_outer_base_knuckle_joint"
-		parent_joint="left_outer_base_knuckle_joint" mimic_joint="right_outer_base_knuckle_joint"
-  	has_pid="true" multiplier="-1.0" max_effort="10.0" />
+    <xacro:mimic_joint_plugin_gazebo name_prefix="right_inner_base_knuckle_joint"
+  		parent_joint="left_outer_base_knuckle_joint" mimic_joint="right_inner_base_knuckle_joint"
+    	has_pid="true" multiplier="-1.0" max_effort="10.0" />
+    <xacro:mimic_joint_plugin_gazebo name_prefix="right_inner_knuckle_finger_joint"
+  		parent_joint="left_outer_base_knuckle_joint" mimic_joint="right_inner_knuckle_finger_joint"
+    	has_pid="true" multiplier="1.0" max_effort="10.0" />
+    <xacro:mimic_joint_plugin_gazebo name_prefix="right_outer_base_knuckle_joint"
+  		parent_joint="left_outer_base_knuckle_joint" mimic_joint="right_outer_base_knuckle_joint"
+    	has_pid="true" multiplier="-1.0" max_effort="10.0" />
 </robot>

File: mycobot_gripper_description/urdf/gripper.urdf.xacro (robot description, xacro)
@@ -5,8 +5,5 @@
 	<xacro:include filename="$(find mycobot_description)/urdf/gripper/gripper.transmission.xacro" />
 	<xacro:include filename="$(find mycobot_description)/urdf/common.xacro" />
-	<material name="white">
-		<color rgba="0.79216 0.81961 0.93333 1" />
-	</material>
-<!-- ============================   Mycobot_Gripper   ============================ -->
+<!-- ============================   Mycobot_Arm   ============================ -->
 	<xacro:macro name="mycobot_gripper" params="parent *origin">
 			<!-- defining the base link -->
@@ -15,5 +12,6 @@
 				<origin xyz="0 -0.018162 0" rpy="1.5708 0 0" />
 				<mass value="0.03237" />
-				<inertia ixx="7.9803E-06" ixy="-3.7162E-08" ixz="4.3435E-07" iyy="1.0337E-05" iyz="3.3485E-07" izz="1.5321E-05" />
+				<inertia
+					ixx="7.9803E-06" ixy="-3.7162E-08" ixz="4.3435E-07" iyy="1.0337E-05" iyz="3.3485E-07" izz="1.5321E-05" />
 			</inertial>
 			<visual>
@@ -22,5 +20,7 @@
 					<mesh filename="package://mycobot_description/meshes/gripper/base_link.STL" />
 				</geometry>
-				<material name="white" />
+				<material name="">
+					<color rgba="0.79216 0.81961 0.93333 1" />
+				</material>
 			</visual>
 			<collision>
@@ -36,5 +36,6 @@
 				<origin xyz="-0.013688 0.0077832 0.01" rpy="0 0 0" />
 				<mass value="0.0027253" />
-				<inertia ixx="2.3883E-07" ixy="1.3724E-07" ixz="5.0465E-14" iyy="4.0216E-07" iyz="-1.3375E-14" izz="3.5516E-07" />
+				<inertia
+					ixx="2.3883E-07" ixy="1.3724E-07" ixz="5.0465E-14" iyy="4.0216E-07" iyz="-1.3375E-14" izz="3.5516E-07" />
 			</inertial>
 			<visual>
@@ -43,5 +44,7 @@
 					<mesh filename="package://mycobot_description/meshes/gripper/left_inner_knuckle_link.STL" />
 				</geometry>
-				<material name="white" />
+				<material name="">
+					<color rgba="0.79216 0.81961 0.93333 1" />
+				</material>
 			</visual>
 			<collision>
@@ -57,5 +60,6 @@
 			<origin xyz="-0.011258 -0.00023581 0.005" rpy="0 0 0" />
 			<mass value="0.0069464" />
-			<inertia ixx="3.0023E-07" ixy="1.5317E-07" ixz="2.0426E-16" iyy="1.5826E-06" iyz="-6.683E-17" izz="1.4568E-06" />
+			<inertia
+				ixx="3.0023E-07" ixy="1.5317E-07" ixz="2.0426E-16" iyy="1.5826E-06" iyz="-6.683E-17" izz="1.4568E-06" />
 		</inertial>
 		<visual>
@@ -64,5 +68,7 @@
 				<mesh filename="package://mycobot_description/meshes/gripper/left_finger_link.STL" />
 			</geometry>
-			<material name="white" />
+			<material name="">
+		    <color rgba="0.79216 0.81961 0.93333 1" />
+		  </material>
 		</visual>
 		<collision>
@@ -87,5 +93,7 @@
 					<mesh filename="package://mycobot_description/meshes/gripper/left_outer_knuckle_link.STL" />
 				</geometry>
-				<material name="white" />
+				<material name="">
+					<color rgba="0.79216 0.81961 0.93333 1" />
+				</material>
 			</visual>
 			<collision>
@@ -108,5 +116,7 @@
 				<mesh filename="package://mycobot_description/meshes/gripper/right_inner_knuckle_link.STL" />
 			</geometry>
-			<material name="white" />
+			<material name="">
+				  <color rgba="0.79216 0.81961 0.93333 1" />
+      </material>
 		</visual>
 		<collision>
@@ -129,5 +139,7 @@
 					<mesh filename="package://mycobot_description/meshes/gripper/right_finger_link.STL" />
 				</geometry>
-				<material name="white" />
+				<material name="">
+					<color rgba="0.79216 0.81961 0.93333 1" />
+		    </material>
 			</visual>
 			<collision>
@@ -150,5 +162,7 @@
 					<mesh filename="package://mycobot_description/meshes/gripper/right_outer_knuckle_link.STL" />
 				</geometry>
-				<material name="white" />
+				<material name="">
+					<color rgba="0.79216 0.81961 0.93333 1" />
+				</material>
 			</visual>
 			<collision>
@@ -159,11 +173,4 @@
 			</collision>
 		</link>
-		<!-- define the grasping frame-->
-		<link name="grasping_frame" />
-		<joint name="grasping_frame_joint" type="fixed">
-			<parent link="gripper_base_link" />
-			<child link="grasping_frame" />
-			<origin rpy="${pi/2} 0 0" xyz="0 -0.0038 0.0533" />
-		</joint>
 		<!-- define the gripper base joint-->
 		<joint name="gripper_base_joint" type="fixed">

File: mycobot_moveit_config/config/gazebo_mycobot.urdf (robot description, URDF)
Before this commit: robot mycobot, 25 links, 24 joints
Links:
- added link grasping_frame
Joints:
- added joint grasping_frame_joint: type fixed, parent gripper_base_link, child grasping_frame, origin xyz=0 -0.0038 0.0533 rpy=1.5707963267948966 0 0
- joint left_inner_base_knuckle_joint: limit (none) -> lower=-3 upper=3 effort=10 velocity=0.05; type continuous -> revolute
- joint left_inner_knuckle_finger_joint: limit (none) -> lower=-3 upper=3 effort=10 velocity=0.05; type continuous -> revolute
- joint right_inner_base_knuckle_joint: limit (none) -> lower=-3 upper=3 effort=10 velocity=0.05; type continuous -> revolute
- joint right_inner_knuckle_finger_joint: limit (none) -> lower=-3 upper=3 effort=10 velocity=0.05; type continuous -> revolute
- joint right_outer_base_knuckle_joint: limit (none) -> lower=-3 upper=3 effort=10 velocity=0.05; type continuous -> revolute
